Commit message: Edit stl file path in urdf file

File: dofbot_ws/src/smart_headlamp_pkg/urdf/dofbot_with_line.urdf (robot description, URDF)
Before this commit: robot dofbot, 4 links, 3 joints
Links:
- link base_link: geometry collision mesh filename=package://smart_headlamp_pkg/meshes/base_link.STL; visual mesh filename=package://smart_headlamp_pkg/meshes/base_link.STL
- link link1: geometry collision mesh filename=package://smart_headlamp_pkg/meshes/link1.STL; visual mesh filename=package://smart_headlamp_pkg/meshes/link1.STL
- link link2: geometry collision mesh filename=package://smart_headlamp_pkg/meshes/link2.STL; visual mesh filename=package://smart_headlamp_pkg/meshes/link2.STL
